Commit message: setting up nav2

File: install/microver_dusty/share/microver_dusty/models/microver.urdf.xacro (robot description, xacro)
@@ -87,5 +87,65 @@
         <child link="front_right_leg_link" />
     </joint>
+                    <!-- ####################### LIDAR SETUP #################### -->
+    <joint name="lidar_joint" type="fixed">
+        <origin xyz="0 0 0.12" rpy="0 0 0" />
+        <parent link="base_link" />
+        <child link="lidar_link" />
+    </joint>
                     <!-- ####################### LINKS ########################## -->
+                     <!-- TODO: EDIT THE RANDOM ASS VALUES IN THE LIDAR LINK -->
+    <link name="lidar_link">
+    <inertial>
+        <origin xyz="0 0 0" rpy="0 0 0"/>
+        <mass value="0.125"/>
+        <inertia ixx="0.001" ixy="0" ixz="0" iyy="0.001" iyz="0" izz="0.001" />
+    </inertial>
+    <collision>
+        <origin xyz="0 0 0" rpy="0 0 0"/>
+        <geometry>
+        <cylinder radius="0.0508" length="0.055"/>
+        </geometry>
+    </collision>
+    <visual>
+        <origin xyz="0 0 0" rpy="0 0 0"/>
+        <geometry>
+        <cylinder radius="0.0508" length="0.055"/>
+        </geometry>
+    </visual>
+    </link>
+    <gazebo reference="lidar_link">
+    <sensor name="lidar" type="ray">
+        <always_on>true</always_on>
+        <visualize>true</visualize>
+        <update_rate>5</update_rate>
+        <ray>
+        <scan>
+            <horizontal>
+            <samples>360</samples>
+            <resolution>1.000000</resolution>
+            <min_angle>0.000000</min_angle>
+            <max_angle>6.280000</max_angle>
+            </horizontal>
+        </scan>
+        <range>
+            <min>0.120000</min>
+            <max>3.5</max>
+            <resolution>0.015000</resolution>
+        </range>
+        <noise>
+            <type>gaussian</type>
+            <mean>0.0</mean>
+            <stddev>0.01</stddev>
+        </noise>
+        </ray>
+        <plugin name="scan" filename="libgazebo_ros_ray_sensor.so">
+        <ros>
+            <remapping>~/out:=scan</remapping>
+        </ros>
+        <output_type>sensor_msgs/LaserScan</output_type>
+        <frame_name>lidar_link</frame_name>
+        </plugin>
+    </sensor>
+    </gazebo>
     <link name="chassis">
         <visual>
@@ -273,3 +333,4 @@
         <mu2 value="${MU2}" />
     </gazebo>
+    <!-- ################## LIDAR  ################### -->
 </robot>
