Commit message: wheels now show up on slam, transform from odom to base link is now dynamic. maybe test with rt2fo later with RPI4B

File: src/roombav2/models/constants.xacro (robot description, xacro)
@@ -4,6 +4,6 @@
     <xacro:property name="MAX_SPEED"    value="5.5"  />
     <xacro:property name="MIN_SPEED"    value="0.0"  />
-    <xacro:property name="WHEEL_RADIUS" value="0.04" />
-    <xacro:property name="WHEEL_WIDTH"  value="0.05"  />
+    <xacro:property name="WHEEL_RADIUS" value="0.06" />
+    <xacro:property name="WHEEL_WIDTH"  value="0.06"  />
     <xacro:property name="WHEELBASE"    value="0.5"  />
     <xacro:property name="WHEEL_MASS"   value="0.45"  />

File: src/roombav2/models/microver.urdf.xacro (robot description, xacro)
@@ -14,7 +14,4 @@
         <color rgba="0.2 0.2 1 1" />
     </material>
-    <material name="purple">
-        <color rgba="0.62 0.12 0.94 1" />
-    </material>
     <!-- the base link located in the middle of the line that goes through the center of both back wheels -->
     <link name="base_link">
@@ -90,5 +87,5 @@
                     <!-- ####################### LIDAR SETUP #################### -->
     <joint name="lidar_joint" type="fixed">
-        <origin xyz="0 0 0.12" rpy="0 0 0" />
+        <origin xyz="0 0 0.168" rpy="0 0 ${pi}" />
         <parent link="base_link" />
         <child link="lidar_link" />
@@ -97,9 +94,4 @@
                      <!-- TODO: EDIT THE RANDOM ASS VALUES IN THE LIDAR LINK -->
     <link name="lidar_link">
-        <inertial>
-            <origin xyz="0 0 0" rpy="0 0 0"/>
-            <mass value="0.125"/>
-            <inertia ixx="0.001" ixy="0" ixz="0" iyy="0.001" iyz="0" izz="0.001" />
-        </inertial>
         <collision>
             <origin xyz="0 0 0" rpy="0 0 0"/>
@@ -205,11 +197,11 @@
                 <cylinder radius="${WHEEL_RADIUS}" length="${WHEEL_WIDTH}" />
             </geometry>
-            <material name="purple" />
-        </visual>
-        <collision>
-            <geometry>
-                <cylinder radius="${WHEEL_RADIUS}" length="${WHEEL_WIDTH}" />
-            </geometry>
-        </collision>
+            <material name="white" />
+        </visual>
+        <!-- <collision>
+            <geometry>
+                <cylinder radius="${WHEEL_RADIUS}" length="${WHEEL_WIDTH}" />
+            </geometry>
+        </collision> -->
         <xacro:inertial_cylinder mass="${WHEEL_MASS}" length="${WHEEL_WIDTH}" radius="${WHEEL_RADIUS}">
             <origin xyz="0 0 0"/>
@@ -221,11 +213,11 @@
                 <cylinder radius="${WHEEL_RADIUS}" length="${WHEEL_WIDTH}" />
             </geometry>
-            <material name="purple" />
-        </visual>
-        <collision>
-            <geometry>
-                <cylinder radius="${WHEEL_RADIUS}" length="${WHEEL_WIDTH}" />
-            </geometry>
-        </collision>
+            <material name="white" />
+        </visual>
+        <!-- <collision>
+            <geometry>
+                <cylinder radius="${WHEEL_RADIUS}" length="${WHEEL_WIDTH}" />
+            </geometry>
+        </collision> -->
         <xacro:inertial_cylinder mass="${WHEEL_MASS}" length="${WHEEL_WIDTH}" radius="${WHEEL_RADIUS}">
             <origin xyz="0 0 0"/>
@@ -237,11 +229,11 @@
                 <cylinder radius="${WHEEL_RADIUS}" length="${WHEEL_WIDTH}" />
             </geometry>
-            <material name="purple" />
-        </visual>
-        <collision>
-            <geometry>
-                <cylinder radius="${WHEEL_RADIUS}" length="${WHEEL_WIDTH}" />
-            </geometry>
-        </collision>
+            <material name="white" />
+        </visual>
+        <!-- <collision>
+            <geometry>
+                <cylinder radius="${WHEEL_RADIUS}" length="${WHEEL_WIDTH}" />
+            </geometry>
+        </collision> -->
         <xacro:inertial_cylinder mass="${WHEEL_MASS}" length="${WHEEL_WIDTH}" radius="${WHEEL_RADIUS}">
             <origin xyz="0 0 0"/>
@@ -253,11 +245,11 @@
                 <cylinder radius="${WHEEL_RADIUS}" length="${WHEEL_WIDTH}" />
             </geometry>
-            <material name="purple" />
-        </visual>
-        <collision>
-            <geometry>
-                <cylinder radius="${WHEEL_RADIUS}" length="${WHEEL_WIDTH}" />
-            </geometry>
-        </collision>
+            <material name="white" />
+        </visual>
+        <!-- <collision>
+            <geometry>
+                <cylinder radius="${WHEEL_RADIUS}" length="${WHEEL_WIDTH}" />
+            </geometry>
+        </collision> -->
         <xacro:inertial_cylinder mass="${WHEEL_MASS}" length="${WHEEL_WIDTH}" radius="${WHEEL_RADIUS}">
             <origin xyz="0 0 0"/>
@@ -281,20 +273,20 @@
     </gazebo>
     <gazebo reference="front_left_wheel_link">
-        <material>Gazebo/Purple</material>
+        <material>Gazebo/white</material>
         <mu1 value="${MU1}" />
         <mu2 value="${MU2}" />
     </gazebo>
     <gazebo reference="front_right_wheel_link">
-        <material>Gazebo/Purple</material>
+        <material>Gazebo/white</material>
         <mu1 value="${MU1}" />
         <mu2 value="${MU2}" />
     </gazebo>
     <gazebo reference="back_left_wheel_link">
-        <material>Gazebo/Purple</material>
+        <material>Gazebo/white</material>
         <mu1 value="${MU1}" />
         <mu2 value="${MU2}" />
     </gazebo>
     <gazebo reference="back_right_wheel_link">
-        <material>Gazebo/Purple</material>
+        <material>Gazebo/white</material>
         <mu1 value="${MU1}" />
         <mu2 value="${MU2}" />
